File: SensorArray.kicad_pcb (KiCad board)
At the start: 2 copper layers, 5 parts

Commit message: More Thinks finished week 7
Parts:
- added SOP65P640X110-24N: VAL**, TCA9548APWR:SOP65P640X110-24N, F.Cu at (95.2, 127.0)
- moved SENSOR_VL53L0X 28.2 mm to (74.9, 134.6)
- moved SENSOR_VL53L0X 26.2 mm to (74.9, 130.8)
- moved SENSOR_VL53L0X 25.0 mm to (74.9, 119.4)
- moved SENSOR_VL53L0X 23.0 mm to (74.9, 127.0)
- moved SENSOR_VL53L0X 22.2 mm to (74.9, 123.2)

Commit message: updated schematic and pcb layout
Parts:
- added SENSOR_VL53L0X: VAL**, VL53L0X:SENSOR_VL53L0X, F.Cu at (74.9, 138.4)

Commit message: pcb made
Parts:
- removed SENSOR_VL53L0X (x6): VAL**, VL53L0X:SENSOR_VL53L0X
- removed SOP65P640X110-24N: VAL**, TCA9548APWR:SOP65P640X110-24N
- added C1: 0.1uf, Capacitor _0.1uf:CAPC0603X33N, F.Cu at (179.0, 80.0)
- added C10: 10uf, 0603-NO:0603-NO, F.Cu at (160.7, 91.4)
- added C11: 10uf, 0603-NO:0603-NO, F.Cu at (163.8, 91.4)
- added C12: 10uf, 0603-NO:0603-NO, F.Cu at (160.7, 86.4)
- added C13: 10uf, 0603-NO:0603-NO, F.Cu at (163.8, 86.4)
- added C14: 10uf, 0603-NO:0603-NO, F.Cu at (160.7, 81.0)
- added C15: 10uf, 0603-NO:0603-NO, F.Cu at (163.8, 81.0)
- added C16: 10uf, 0603-NO:0603-NO, F.Cu at (172.7, 86.4)
- added C17: 10uf, 0603-NO:0603-NO, F.Cu at (172.7, 91.4)
- added C18: 10uf, 0603-NO:0603-NO, F.Cu at (175.3, 86.4)
- added C19: 10uf, 0603-NO:0603-NO, F.Cu at (175.3, 91.4)
- added C2: 0.1uf, Capacitor _0.1uf:CAPC0603X33N, F.Cu at (179.0, 82.5)
- added C3: 0.1uf, Capacitor _0.1uf:CAPC0603X33N, F.Cu at (179.0, 85.1)
- added C4: 0.1uf, Capacitor _0.1uf:CAPC0603X33N, F.Cu at (179.0, 87.6)
- added C5: 0.1uf, Capacitor _0.1uf:CAPC0603X33N, F.Cu at (179.0, 90.2)
- added C6: 0.1uf, Capacitor _0.1uf:CAPC0603X33N, F.Cu at (179.0, 92.7)
- added C7: 10uf, 0603-NO:0603-NO, F.Cu at (151.8, 87.0)
- added C8: 10uf, 0603-NO:0603-NO, F.Cu at (175.3, 81.3)
- added C9: 10uf, 0603-NO:0603-NO, F.Cu at (172.7, 81.3)
- added IC1: MIC1, MIC5225-5.0YM5-TR:SOT95P280X130-5N, F.Cu at (168.3, 81.3)
- added IC2: MIC6, MIC5225-5.0YM5-TR:SOT95P280X130-5N, F.Cu at (156.2, 91.4)
- added IC3: MIC5, MIC5225-5.0YM5-TR:SOT95P280X130-5N, F.Cu at (156.2, 86.4)
- added IC4: MIC4, MIC5225-5.0YM5-TR:SOT95P280X130-5N, F.Cu at (156.2, 81.0)
- added IC5: MIC2, MIC5225-5.0YM5-TR:SOT95P280X130-5N, F.Cu at (168.3, 86.4)
- added IC6: MIC3, MIC5225-5.0YM5-TR:SOT95P280X130-5N, F.Cu at (168.3, 91.4)
- added J1: Conn_01x08, Connector_PinSocket_2.54mm:PinSocket_1x08_P2.54mm_Vertical, F.Cu at (133.3, 94.0)
- added JP1: , Jumper:SolderJumper-2_P1.3mm_Open_Pad1.0x1.5mm, F.Cu at (138.4, 81.3)
- added JP2: , Jumper:SolderJumper-2_P1.3mm_Open_Pad1.0x1.5mm, F.Cu at (138.4, 76.2)
- added JP3: SolderJumper_2_Open, Jumper:SolderJumper-2_P1.3mm_Open_Pad1.0x1.5mm, F.Cu at (138.4, 86.4)
- added JP4: SolderJumper_2_Open, Jumper:SolderJumper-2_P1.3mm_Open_Pad1.0x1.5mm, F.Cu at (142.2, 94.6)
- added JP5: SolderJumper_2_Open, Jumper:SolderJumper-2_P1.3mm_Open_Pad1.0x1.5mm, F.Cu at (138.4, 91.4)
- added Q1: BSS138, Package_TO_SOT_SMD:SOT-23, F.Cu at (151.3, 97.1)
- added Q10: BSS138, Package_TO_SOT_SMD:SOT-23, F.Cu at (178.2, 97.2)
- added Q11: BSS138, Package_TO_SOT_SMD:SOT-23, F.Cu at (190.0, 74.7)
- added Q12: BSS138, Package_TO_SOT_SMD:SOT-23, F.Cu at (189.7, 91.5)
- added Q2: BSS138, Package_TO_SOT_SMD:SOT-23, F.Cu at (159.2, 96.9)
- added Q3: BSS138, Package_TO_SOT_SMD:SOT-23, F.Cu at (189.7, 86.8)
- added Q4: BSS138, Package_TO_SOT_SMD:SOT-23, F.Cu at (189.7, 82.3)
- added Q5: BSS138, Package_TO_SOT_SMD:SOT-23, F.Cu at (146.7, 79.1)
- added Q6: BSS138, Package_TO_SOT_SMD:SOT-23, F.Cu at (146.5, 74.7)
- added Q7: BSS138, Package_TO_SOT_SMD:SOT-23, F.Cu at (168.2, 97.3)
- added Q8: BSS138, Package_TO_SOT_SMD:SOT-23, F.Cu at (190.0, 78.2)
- added Q9: BSS138, Package_TO_SOT_SMD:SOT-23, F.Cu at (189.7, 95.3)
- added R1: 10k, RESC0603X26N:RESC0603X26N, F.Cu at (181.2, 80.0)
- added R10: 10k, RESC0603X26N:RESC0603X26N, F.Cu at (182.9, 92.7)
- added R11: 10k, RESC0603X26N:RESC0603X26N, F.Cu at (181.3, 92.7)
- added R12: 10k, RESC0603X26N:RESC0603X26N, F.Cu at (151.8, 84.5)
- added R13: 10k, RESC0603X26N:RESC0603X26N, F.Cu at (151.8, 79.4)
- added R14: 10k, RESC0603X26N:RESC0603X26N, F.Cu at (151.8, 81.9)
- added R15: 10k, RESC0603X26N:RESC0603X26N, F.Cu at (181.3, 85.1)
- added R16: 10k, RESC0603X26N:RESC0603X26N, F.Cu at (147.1, 97.1)
- added R17: 10k, RESC0603X26N:RESC0603X26N, F.Cu at (163.0, 96.9)
- added R18: 10k, RESC0603X26N:RESC0603X26N, F.Cu at (151.8, 89.5)
- added R19: 10k, RESC0603X26N:RESC0603X26N, F.Cu at (146.4, 94.0)
- added R2: 10k, RESC0603X26N:RESC0603X26N, F.Cu at (182.9, 80.0)
- added R20: 10k, RESC0603X26N:RESC0603X26N, F.Cu at (149.9, 94.0)
- added R21: 10k, RESC0603X26N:RESC0603X26N, F.Cu at (154.1, 97.1)
- added R22: 10k, RESC0603X26N:RESC0603X26N, F.Cu at (156.6, 96.9)
- added R23: 10k, RESC0603X26N:RESC0603X26N, F.Cu at (185.9, 86.8)
- added R24: 10k, RESC0603X26N:RESC0603X26N, F.Cu at (185.9, 82.3)
- added R25: 10k, RESC0603X26N:RESC0603X26N, F.Cu at (192.2, 86.8)
- added R26: 10k, RESC0603X26N:RESC0603X26N, F.Cu at (192.5, 82.3)
- added R27: 10k, RESC0603X26N:RESC0603X26N, F.Cu at (142.0, 79.4)
- added R28: 10k, RESC0603X26N:RESC0603X26N, F.Cu at (142.2, 74.9)
- added R29: 10k, RESC0603X26N:RESC0603X26N, F.Cu at (149.5, 79.1)
- added R3: 10k, RESC0603X26N:RESC0603X26N, F.Cu at (182.9, 82.5)
- added R30: 10k, RESC0603X26N:RESC0603X26N, F.Cu at (149.4, 74.7)
- added R31: 10k, RESC0603X26N:RESC0603X26N, F.Cu at (172.0, 97.3)
- added R32: 10k, RESC0603X26N:RESC0603X26N, F.Cu at (185.7, 78.2)
- added R33: 10k, RESC0603X26N:RESC0603X26N, F.Cu at (185.9, 95.3)
- added R34: 10k, RESC0603X26N:RESC0603X26N, F.Cu at (174.4, 97.2)
- added R35: 10k, RESC0603X26N:RESC0603X26N, F.Cu at (185.8, 74.7)
- added R36: 10k, RESC0603X26N:RESC0603X26N, F.Cu at (185.9, 91.5)
- added R37: 10k, RESC0603X26N:RESC0603X26N, F.Cu at (165.6, 97.3)
- added R38: 10k, RESC0603X26N:RESC0603X26N, F.Cu at (192.8, 78.2)
- added R39: 10k, RESC0603X26N:RESC0603X26N, F.Cu at (192.5, 95.3)
- added R4: 10k, RESC0603X26N:RESC0603X26N, F.Cu at (181.3, 82.5)
- added R40: 10k, RESC0603X26N:RESC0603X26N, F.Cu at (181.1, 97.2)
- added R41: 10k, RESC0603X26N:RESC0603X26N, F.Cu at (192.8, 74.9)
- added R42: 10k, RESC0603X26N:RESC0603X26N, F.Cu at (192.7, 91.5)
- added R5: 10k, RESC0603X26N:RESC0603X26N, F.Cu at (182.9, 85.1)
- added R6: 10k, RESC0603X26N:RESC0603X26N, F.Cu at (182.9, 87.6)
- added R7: 10k, RESC0603X26N:RESC0603X26N, F.Cu at (181.3, 87.6)
- added R8: 10k, RESC0603X26N:RESC0603X26N, F.Cu at (182.9, 90.2)
- added R9: 10k, RESC0603X26N:RESC0603X26N, F.Cu at (181.3, 90.2)
- added U1: VL53L0X, VL53L0X:SENSOR_VL53L0X, F.Cu at (165.7, 74.8)
- added U2: TCA9548APWR, Package_SO:TSSOP-24_4.4x7.8mm_P0.65mm, F.Cu at (146.1, 87.0)
- added U3: VL53L0X, VL53L0X:SENSOR_VL53L0X, F.Cu at (177.2, 74.8)
- added U4: VL53L0X, VL53L0X:SENSOR_VL53L0X, F.Cu at (161.6, 74.8)
- added U5: VL53L0X, VL53L0X:SENSOR_VL53L0X, F.Cu at (173.4, 74.8)
- added U6: VL53L0X, VL53L0X:SENSOR_VL53L0X, F.Cu at (157.5, 74.8)
- added U7: VL53L0X, VL53L0X:SENSOR_VL53L0X, F.Cu at (169.5, 74.8)
Routing:
- net GND: track 0.00 -> 245.2 mm, vias 0 -> 4
- net VCC: track 0.00 -> 223.8 mm, vias 0 -> 2
- net /OUT_3: track 0.00 -> 105.0 mm, vias 0 -> 3
- net /OUT_2: track 0.00 -> 83.3 mm, vias 0 -> 3
- net /OUT_5: track 0.00 -> 83.1 mm, vias 0 -> 4
- net /OUT_1: track 0.00 -> 75.3 mm, vias 0 -> 4
- net /SD0: track 0.00 -> 73.4 mm, vias 0 -> 4
- net Net-(R3-Pad2): track 0.00 -> 69.9 mm, vias 0 -> 2
- net /OUT_4: track 0.00 -> 69.4 mm, vias 0 -> 2
- net /SC2_2.8: track 0.00 -> 66.3 mm, vias 0 -> 2
- net /SC1: track 0.00 -> 63.2 mm, vias 0 -> 2
- net /SD1: track 0.00 -> 63.1 mm, vias 0 -> 2
- net /SC4: track 0.00 -> 62.0 mm, vias 0 -> 2
- net /SC0: track 0.00 -> 61.8 mm, vias 0 -> 2
- net /SD4: track 0.00 -> 61.4 mm, vias 0 -> 2
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Other:
- board outline added: 67.3 x 31.1 mm
- board text added: "Christian Silver Cedric Fely Zhiying HP Mathmatica"
