File: SensorArray.sch (KiCad schematic (older format))
At the start: 6 parts

Commit message: Week 6 Progress
Parts:
- added R? (x6): R, symbol device:R
- added U?: TCA9548APWR, SOP65P640X110-24N, symbol TCA9548APWR:TCA9548APWR
Connections:
- net at U?.5 (~XSHUT~): now also R?.2 (x3)
- net at U?.7 (GPIO1): now also R?.2 (x2)
Other:
- moved on the sheet: U?
Changed lines of the file:
@@
 L VL53L0X:VL53L0X U?
 U 1 1 5BE62F63
-P 10000 4050
-F 0 "U?" H 10000 4715 50  0000 C CNN
-F 1 "VL53L0X" H 10000 4624 50  0000 C CNN
-F 2 "SENSOR_VL53L0X" H 10000 4050 50  0001 L BNN
-F 3 "STMicroelectronics" H 10000 4050 50  0001 L BNN
-F 4 "World smallest Time-of-Flight _ToF_ ranging sensor" H 10000 4050 50  0001 L BNN "Field4"
-F 5 "None" H 10000 4050 50  0001 L BNN "Field5"
-F 6 "VL53L0X" H 10000 4050 50  0001 L BNN "Field6"
-F 7 "Unavailable" H 10000 4050 50  0001 L BNN "Field7"
-F 8 "None" H 10000 4050 50  0001 L BNN "Field8"
-	1    10000 4050
+P 9800 1750
+F 0 "U?" H 9800 2415 50  0000 C CNN
+F 1 "VL53L0X" H 9800 2324 50  0000 C CNN
+F 2 "SENSOR_VL53L0X" H 9800 1750 50  0001 L BNN
+F 3 "STMicroelectronics" H 9800 1750 50  0001 L BNN
+F 4 "World smallest Time-of-Flight _ToF_ ranging sensor" H 9800 1750 50  0001 L BNN "Field4"
+F 5 "None" H 9800 1750 50  0001 L BNN "Field5"
+F 6 "VL53L0X" H 9800 1750 50  0001 L BNN "Field6"
+F 7 "Unavailable" H 9800 1750 50  0001 L BNN "Field7"
+F 8 "None" H 9800 1750 50  0001 L BNN "Field8"
+	1    9800 1750
 	1    0    0    -1
 $EndComp
@@
 L VL53L0X:VL53L0X U?
 U 1 1 5BE631E4
-P 8450 4050
-F 0 "U?" H 8450 4715 50  0000 C CNN
-F 1 "VL53L0X" H 8450 4624 50  0000 C CNN
-F 2 "SENSOR_VL53L0X" H 8450 4050 50  0001 L BNN
-F 3 "STMicroelectronics" H 8450 4050 50  0001 L BNN
-F 4 "World smallest Time-of-Flight _ToF_ ranging sensor" H 8450 4050 50  0001 L BNN "Field4"
-F 5 "None" H 8450 4050 50  0001 L BNN "Field5"
-F 6 "VL53L0X" H 8450 4050 50  0001 L BNN "Field6"
-F 7 "Unavailable" H 8450 4050 50  0001 L BNN "Field7"
-F 8 "None" H 8450 4050 50  0001 L BNN "Field8"
-	1    8450 4050
+P 7900 1750
+F 0 "U?" H 7900 2415 50  0000 C CNN
+F 1 "VL53L0X" H 7900 2324 50  0000 C CNN
+F 2 "SENSOR_VL53L0X" H 7900 1750 50  0001 L BNN
+F 3 "STMicroelectronics" H 7900 1750 50  0001 L BNN
+F 4 "World smallest Time-of-Flight _ToF_ ranging sensor" H 7900 1750 50  0001 L BNN "Field4"
+F 5 "None" H 7900 1750 50  0001 L BNN "Field5"
+F 6 "VL53L0X" H 7900 1750 50  0001 L BNN "Field6"
+F 7 "Unavailable" H 7900 1750 50  0001 L BNN "Field7"
+F 8 "None" H 7900 1750 50  0001 L BNN "Field8"
+	1    7900 1750
 	1    0    0    -1
 $EndComp
@@
 L VL53L0X:VL53L0X U?
 U 1 1 5BE6321A
-P 5200 4050
-F 0 "U?" H 5200 4715 50  0000 C CNN
-F 1 "VL53L0X" H 5200 4624 50  0000 C CNN
-F 2 "SENSOR_VL53L0X" H 5200 4050 50  0001 L BNN
-F 3 "STMicroelectronics" H 5200 4050 50  0001 L BNN
-F 4 "World smallest Time-of-Flight _ToF_ ranging sensor" H 5200 4050 50  0001 L BNN "Field4"
-F 5 "None" H 5200 4050 50  0001 L BNN "Field5"
-F 6 "VL53L0X" H 5200 4050 50  0001 L BNN "Field6"
-F 7 "Unavailable" H 5200 4050 50  0001 L BNN "Field7"
-F 8 "None" H 5200 4050 50  0001 L BNN "Field8"
-	1    5200 4050
+P 7800 3800
+F 0 "U?" H 7800 4465 50  0000 C CNN
+F 1 "VL53L0X" H 7800 4374 50  0000 C CNN
+F 2 "SENSOR_VL53L0X" H 7800 3800 50  0001 L BNN
+F 3 "STMicroelectronics" H 7800 3800 50  0001 L BNN
+F 4 "World smallest Time-of-Flight _ToF_ ranging sensor" H 7800 3800 50  0001 L BNN "Field4"
+F 5 "None" H 7800 3800 50  0001 L BNN "Field5"
+F 6 "VL53L0X" H 7800 3800 50  0001 L BNN "Field6"
+F 7 "Unavailable" H 7800 3800 50  0001 L BNN "Field7"
+F 8 "None" H 7800 3800 50  0001 L BNN "Field8"
+	1    7800 3800
 	1    0    0    -1
 $EndComp
@@
 L VL53L0X:VL53L0X U?
 U 1 1 5BE6324A
-P 1800 4000
-F 0 "U?" H 1800 4665 50  0000 C CNN
-F 1 "VL53L0X" H 1800 4574 50  0000 C CNN
-F 2 "SENSOR_VL53L0X" H 1800 4000 50  0001 L BNN
-F 3 "STMicroelectronics" H 1800 4000 50  0001 L BNN
-F 4 "World smallest Time-of-Flight _ToF_ ranging sensor" H 1800 4000 50  0001 L BNN "Field4"
-F 5 "None" H 1800 4000 50  0001 L BNN "Field5"
-F 6 "VL53L0X" H 1800 4000 50  0001 L BNN "Field6"
-F 7 "Unavailable" H 1800 4000 50  0001 L BNN "Field7"
-F 8 "None" H 1800 4000 50  0001 L BNN "Field8"
-	1    1800 4000
+P 2100 1700
+F 0 "U?" H 2100 2365 50  0000 C CNN
+F 1 "VL53L0X" H 2100 2274 50  0000 C CNN
+F 2 "SENSOR_VL53L0X" H 2100 1700 50  0001 L BNN
+F 3 "STMicroelectronics" H 2100 1700 50  0001 L BNN
+F 4 "World smallest Time-of-Flight _ToF_ ranging sensor" H 2100 1700 50  0001 L BNN "Field4"
+F 5 "None" H 2100 1700 50  0001 L BNN "Field5"
+F 6 "VL53L0X" H 2100 1700 50  0001 L BNN "Field6"
+F 7 "Unavailable" H 2100 1700 50  0001 L BNN "Field7"
+F 8 "None" H 2100 1700 50  0001 L BNN "Field8"
+	1    2100 1700
 	1    0    0    -1
 $EndComp
@@
 L VL53L0X:VL53L0X U?
 U 1 1 5BE6329C
-P 3500 4050
-F 0 "U?" H 3500 4715 50  0000 C CNN
-F 1 "VL53L0X" H 3500 4624 50  0000 C CNN
-F 2 "SENSOR_VL53L0X" H 3500 4050 50  0001 L BNN
-F 3 "STMicroelectronics" H 3500 4050 50  0001 L BNN
-F 4 "World smallest Time-of-Flight _ToF_ ranging sensor" H 3500 4050 50  0001 L BNN "Field4"
-F 5 "None" H 3500 4050 50  0001 L BNN "Field5"
-F 6 "VL53L0X" H 3500 4050 50  0001 L BNN "Field6"
-F 7 "Unavailable" H 3500 4050 50  0001 L BNN "Field7"
-F 8 "None" H 3500 4050 50  0001 L BNN "Field8"
-	1    3500 4050
+P 4550 1700
+F 0 "U?" H 4550 2365 50  0000 C CNN
+F 1 "VL53L0X" H 4550 2274 50  0000 C CNN
+F 2 "SENSOR_VL53L0X" H 4550 1700 50  0001 L BNN
+F 3 "STMicroelectronics" H 4550 1700 50  0001 L BNN
+F 4 "World smallest Time-of-Flight _ToF_ ranging sensor" H 4550 1700 50  0001 L BNN "Field4"
+F 5 "None" H 4550 1700 50  0001 L BNN "Field5"
+F 6 "VL53L0X" H 4550 1700 50  0001 L BNN "Field6"
+F 7 "Unavailable" H 4550 1700 50  0001 L BNN "Field7"
+F 8 "None" H 4550 1700 50  0001 L BNN "Field8"
+	1    4550 1700
 	1    0    0    -1
 $EndComp
@@
 L VL53L0X:VL53L0X U?
 U 1 1 5BE632E4
-P 6850 4050
-F 0 "U?" H 6850 4715 50  0000 C CNN
-F 1 "VL53L0X" H 6850 4624 50  0000 C CNN
-F 2 "SENSOR_VL53L0X" H 6850 4050 50  0001 L BNN
-F 3 "STMicroelectronics" H 6850 4050 50  0001 L BNN
-F 4 "World smallest Time-of-Flight _ToF_ ranging sensor" H 6850 4050 50  0001 L BNN "Field4"
-F 5 "None" H 6850 4050 50  0001 L BNN "Field5"
-F 6 "VL53L0X" H 6850 4050 50  0001 L BNN "Field6"
-F 7 "Unavailable" H 6850 4050 50  0001 L BNN "Field7"
-F 8 "None" H 6850 4050 50  0001 L BNN "Field8"
-	1    6850 4050
+P 9800 3850
+F 0 "U?" H 9800 4515 50  0000 C CNN
+F 1 "VL53L0X" H 9800 4424 50  0000 C CNN
+F 2 "SENSOR_VL53L0X" H 9800 3850 50  0001 L BNN
+F 3 "STMicroelectronics" H 9800 3850 50  0001 L BNN
+F 4 "World smallest Time-of-Flight _ToF_ ranging sensor" H 9800 3850 50  0001 L BNN "Field4"
+F 5 "None" H 9800 3850 50  0001 L BNN "Field5"
+F 6 "VL53L0X" H 9800 3850 50  0001 L BNN "Field6"
+F 7 "Unavailable" H 9800 3850 50  0001 L BNN "Field7"
+F 8 "None" H 9800 3850 50  0001 L BNN "Field8"
+	1    9800 3850
 	1    0    0    -1
 $EndComp
+$Comp
+L device:R R?
+U 1 1 5BE64531
+P 3050 1400
+F 0 "R?" H 3120 1446 50  0000 L CNN
+F 1 "R" H 3120 1355 50  0000 L CNN
+F 2 "" V 2980 1400 50  0001 C CNN
+F 3 "" H 3050 1400 50  0001 C CNN
+	1    3050 1400
+	1    0    0    -1
+$EndComp
+$Comp
+L device:R R?
+U 1 1 5BE647CB
+P 1250 1400
+F 0 "R?" H 1320 1446 50  0000 L CNN
+F 1 "R" H 1320 1355 50  0000 L CNN
+F 2 "" V 1180 1400 50  0001 C CNN
+F 3 "" H 1250 1400 50  0001 C CNN
+	1    1250 1400
+	1    0    0    -1
+$EndComp
+Wire Wire Line
+	1400 1600 1250 1600
+Wire Wire Line
+	1250 1600 1250 1550
+$Comp
+L device:R R?
+U 1 1 5BE64CCC
+P 3850 1300
+F 0 "R?" H 3920 1346 50  0000 L CNN
+F 1 "R" H 3920 1255 50  0000 L CNN
+F 2 "" V 3780 1300 50  0001 C CNN
+F 3 "" H 3850 1300 50  0001 C CNN
+	1    3850 1300
+	1    0    0    -1
+$EndComp
+$Comp
+L device:R R?
+U 1 1 5BE64D4A
+P 5550 1350
+F 0 "R?" H 5620 1396 50  0000 L CNN
+F 1 "R" H 5620 1305 50  0000 L CNN
+F 2 "" V 5480 1350 50  0001 C CNN
+F 3 "" H 5550 1350 50  0001 C CNN
+	1    5550 1350
+	1    0    0    -1
+$EndComp
+Wire Wire Line
+	3850 1450 3850 1600
+$Comp
+L device:R R?
+U 1 1 5BE660F3
+P 7200 1350
+F 0 "R?" H 7270 1396 50  0000 L CNN
+F 1 "R" H 7270 1305 50  0000 L CNN
+F 2 "" V 7130 1350 50  0001 C CNN
+F 3 "" H 7200 1350 50  0001 C CNN
+	1    7200 1350
+	1    0    0    -1
+$EndComp
+$Comp
+L device:R R?
+U 1 1 5BE6624D
+P 6950 1350
+F 0 "R?" H 7020 1396 50  0000 L CNN
+F 1 "R" H 7020 1305 50  0000 L CNN
+F 2 "" V 6880 1350 50  0001 C CNN
+F 3 "" H 6950 1350 50  0001 C CNN
+	1    6950 1350
+	1    0    0    -1
+$EndComp
+$Comp
+L TCA9548APWR:TCA9548APWR U?
+U 1 1 5BE665CC
+P 3650 5100
+F 0 "U?" H 3650 5100 50  0001 L BNN
+F 1 "TCA9548APWR" H 3650 5100 50  0001 L BNN
+F 2 "SOP65P640X110-24N" H 3650 5100 50  0001 L BNN
+F 3 "Unavailable" H 3650 5100 50  0001 L BNN
+F 4 "TSSOP-24 Texas Instruments" H 3650 5100 50  0001 L BNN "Field4"
+F 5 "None" H 3650 5100 50  0001 L BNN "Field5"
+F 6 "TCA9548APWR" H 3650 5100 50  0001 L BNN "Field6"
+F 7 "Low-Voltage 8-Channel I2C Switch With Reset 24-TSSOP -40 to 85" H 3650 5100 50  0001 L BNN "Field7"
+F 8 "Texas Instruments" H 3650 5100 50  0001 L BNN "Field8"
+	1    3650 5100
+	1    0    0    -1
+$EndComp
+Wire Wire Line
+	3050 1550 3050 1600
+Wire Wire Line
+	3050 1600 2800 1600
+Wire Wire Line
+	7200 1500 7200 1650
+Wire Wire Line
+	5250 1600 5550 1600
+Wire Wire Line
+	5550 1600 5550 1500
 $EndSCHEMATC

Commit message: Week 6 Progress
Parts:
- added R? (x6): R, symbol device:R
Connections:
- net at U?.5 (~XSHUT~): now also R?.2 (x3)
- net at U?.7 (GPIO1): now also R?.2 (x4)
- net GND: now reaches U?.12 (GND), U?.3 (GND), U?.4 (GND), U?.6 (GND)
- net GND: now also U?.12 (GND), U?.3 (GND), U?.4 (GND), U?.6 (GND)
Other:
- moved on the sheet: R?, U?

Commit message: More Thinks finished week 7
Parts:
- removed R? (x10): R, symbol device:R
- removed U? (x5): VL53L0X, SENSOR_VL53L0X, symbol VL53L0X:VL53L0X
- added C? (x6): 0.1uf, symbol device:C_Small
- added R? (x10): 10k, symbol device:R
- added U? (x5): VL53L0X, SENSOR_VL53L0X, symbol VL53L0X:VL53L0X
- R1, R2: renamed from R?; value R -> 10k
Connections:
- net labels added: +2V8, SC0, SC1, SC2, SC3, SC4, SC5, SD0, SD1, SD2, SD3, SD4, SD5
- wire segments 26 -> 126
Other:
- moved on the sheet: R1, R2, U?

Commit message: updated schematic and pcb layout
Parts:
- added C7: 10uf, symbol device:C_Small
- added J1, J2: Conn_01x12, symbol Connector:Conn_01x12
- added R12: 10k, symbol device:R
- gave numbers to parts that had none: 15
Connections:
- net labels added: A0, A1, A2, GND_Connect, Reset, SC_IN, SD_IN, VCC
- wire segments 126 -> 166
Other:
- moved on the sheet: C1, C2, C3, C5, C6, R1, R10, R11, R2, R3, R4, R5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

Commit message: pcb made
Parts:
- removed J1, J2: Conn_01x12, symbol Connector:Conn_01x12
- removed U?: TCA9548APWR, SOP65P640X110-24N, symbol TCA9548APWR:TCA9548APWR
- added C10, C11, C12, C13, C14, C15, C16, C17, C18, C19, C8, C9: 10uf, 0603-NO:0603-NO, symbol Device:C_Small
- added IC1, IC2, IC3, IC4, IC5, IC6: MIC5225-5.0YM5-TR, MIC5225-5.0YM5-TR:SOT95P280X130-5N, symbol MIC5225-5.0YM5-TR:MIC5225-5.0YM5-TR
- added J1: Conn_01x08, Connector_PinSocket_2.54mm:PinSocket_1x08_P2.54mm_Vertical, symbol Connector_Generic:Conn_01x08
- added JP1, JP2, JP3, JP4, JP5: SolderJumper_2_Open, Jumper:SolderJumper-2_P1.3mm_Open_Pad1.0x1.5mm, symbol Jumper:SolderJumper_2_Open
- added Q1, Q10, Q11, Q12, Q2, Q3, Q4, Q5, Q6, Q7, Q8, Q9: BSS138, Package_TO_SOT_SMD:SOT-23, symbol Transistor_FET:BSS138
- added R13, R14, R16, R17, R18, R19, R20, R21, R22, R23, R24, R25, R26, R27, R28, R29, R30, R31, R32, R33, R34, R35, R36, R37, R38, R39, R40, R41, R42: 10k, RESC0603X26N:RESC0603X26N, symbol Device:R
- added U2: TCA9548APWR, Package_SO:TSSOP-24_4.4x7.8mm_P0.65mm, symbol Interface_Expansion:TCA9548APWR
- C1, C2, C3, C4, C5, C6: footprint (none) -> Capacitor _0.1uf:CAPC0603X33N; symbol device:C_Small -> SensorArray-rescue:C_Small-device
- C7: footprint (none) -> 0603-NO:0603-NO; symbol device:C_Small -> SensorArray-rescue:C_Small-device
- R1, R10, R11, R12, R2, R3, R4, R5, R6, R7, R8, R9: footprint (none) -> RESC0603X26N:RESC0603X26N; symbol device:R -> SensorArray-rescue:R-device
- R15: renamed from R6; footprint (none) -> RESC0603X26N:RESC0603X26N; symbol device:R -> SensorArray-rescue:R-device
- U1, U3, U4, U5, U6, U7: renamed from U?; footprint SENSOR_VL53L0X -> VL53L0X:SENSOR_VL53L0X; symbol VL53L0X:VL53L0X -> SensorArray-rescue:VL53L0X-VL53L0X
Connections:
- net A0: now also J1.6 (Pin_6), JP3.2 (B), R18.1, U2.21 (A2)
- net A1: now also J1.7 (Pin_7), JP4.2 (B), R20.1, U2.2 (A1)
- net A2: now also J1.8 (Pin_8), JP5.1 (A), R19.1, U2.1 (A0)
- net GND: now also C10.2, C11.2, C12.2, C13.2, C14.2, C15.2, C16.2, C17.2, C18.2, C19.2, C8.2, C9.2, IC1.2 (GND), IC2.2 (GND), IC3.2 (GND), IC4.2 (GND), IC5.2 (GND), IC6.2 (GND), J1.2 (Pin_2), R18.2, R19.2, R20.2, U2.12 (GND)
- net Reset: now also J1.5 (Pin_5), U2.3 (~RESET)
- net SC0: now also Q11.3 (D), R41.2, U2.4 (SD0); no longer U3.10 (SCL)
- net SC1: now also Q12.3 (D), R42.2, U2.6 (SD1); no longer U5.10 (SCL)
- net SC2: now also Q10.3 (D), R40.2, U2.8 (SD2); no longer U7.10 (SCL)
- net SC3: now also Q6.3 (D), R30.2, U2.10 (SD3); no longer U1.10 (SCL)
- net SC4: now also Q4.3 (D), R26.2, U2.13 (SD4); no longer U4.10 (SCL)
- net SC5: now also Q2.3 (D), R22.2, U2.15 (SD5); no longer U6.10 (SCL)
- net SC_IN: now also J1.4 (Pin_4), JP2.2 (B), U2.23 (SDA)
- net SD0: now also Q8.3 (D), R38.2, U2.5 (SC0); no longer U3.9 (SDA)
- net SD1: now also Q9.3 (D), R39.2, U2.7 (SC1); no longer U5.9 (SDA)
- net SD2: now also Q7.3 (D), R37.2, U2.9 (SC2); no longer U7.9 (SDA)
- net SD3: now also Q5.3 (D), R29.2, U2.11 (SC3); no longer U1.9 (SDA)
- net SD4: now also Q3.3 (D), R25.2, U2.14 (SC4); no longer U4.9 (SDA)
- net SD5: now also Q1.3 (D), R21.2, U2.16 (SC5); no longer U6.9 (SDA)
- net SD_IN: now also J1.3 (Pin_3), JP1.2 (B), U2.22 (SCL)
- net VCC: now also C10.1, C12.1, C14.1, C16.1, C17.1, C8.1, IC1.1 (IN), IC1.3 (EN), IC2.1 (IN), IC2.3 (EN), IC3.1 (IN), IC3.3 (EN), IC4.1 (IN), IC4.3 (EN), IC5.1 (IN), IC5.3 (EN), IC6.1 (IN), IC6.3 (EN), J1.1 (Pin_1), JP3.1 (A), JP4.1 (A), JP5.2 (B), R13.1, R14.1, R21.1, R22.1, R25.1, R26.1, R29.1, R30.1, R37.1, R38.1, R39.1, R40.1, R41.1, R42.1, U2.24 (VCC)
- removed net +2V8: C1.1, C2.1, C3.1, C4.1, C5.1, C6.1, R1.1, R10.1, R11.1, R15.1, R2.1, R3.1, R4.1, R5.1, R6.1, R7.1, R8.1, R9.1, U1.1 (AVDDVCSEL), U1.11 (AVDD), U3.1 (AVDDVCSEL), U3.11 (AVDD), U4.1 (AVDDVCSEL), U4.11 (AVDD), U5.1 (AVDDVCSEL), U5.11 (AVDD), U6.1 (AVDDVCSEL), U6.11 (AVDD), U7.1 (AVDDVCSEL), U7.11 (AVDD)
- new net: JP1.1 (A), R13.2
- new net: JP2.1 (A), R14.2
- new net OUT_0: C1.1, C9.1, IC1.5 (OUT), Q11.1 (G), Q8.1 (G), R1.1, R2.1, R32.1, R35.1, U3.1 (AVDDVCSEL), U3.11 (AVDD)
- new net OUT_1: C18.1, C2.1, IC5.5 (OUT), Q12.1 (G), Q9.1 (G), R3.1, R33.1, R36.1, R4.1, U5.1 (AVDDVCSEL), U5.11 (AVDD)
- new net OUT_2: C19.1, C3.1, IC6.5 (OUT), Q10.1 (G), Q7.1 (G), R15.1, R31.1, R34.1, R5.1, U7.1 (AVDDVCSEL), U7.11 (AVDD)
- new net OUT_3: C15.1, C4.1, IC4.5 (OUT), Q5.1 (G), Q6.1 (G), R27.1, R28.1, R6.1, R7.1, U1.1 (AVDDVCSEL), U1.11 (AVDD)
- new net OUT_4: C13.1, C5.1, IC3.5 (OUT), Q3.1 (G), Q4.1 (G), R23.1, R24.1, R8.1, R9.1, U4.1 (AVDDVCSEL), U4.11 (AVDD)
- new net OUT_5: C11.1, C6.1, IC2.5 (OUT), Q1.1 (G), Q2.1 (G), R10.1, R11.1, R16.1, R17.1, U6.1 (AVDDVCSEL), U6.11 (AVDD)
- new net SC0_2.8: Q11.2 (S), R35.2, U3.10 (SCL)
- new net SC1_2.8: Q12.2 (S), R36.2, U5.10 (SCL)
- new net SC2_2.8: Q10.2 (S), R34.2, U7.10 (SCL)
- new net SC3_2.8: Q6.2 (S), R28.2, U1.10 (SCL)
- new net SC4_2.8: Q4.2 (S), R24.2, U4.10 (SCL)
- new net SC5_2.8: Q2.2 (S), R17.2, U6.10 (SCL)
- new net SD0_2.8: Q8.2 (S), R32.2, U3.9 (SDA)
- new net SD1_2.8: Q9.2 (S), R33.2, U5.9 (SDA)
- new net SD2_2.8: Q7.2 (S), R31.2, U7.9 (SDA)
- new net SD3_2.8: Q5.2 (S), R27.2, U1.9 (SDA)
- new net SD4_2.8: Q3.2 (S), R23.2, U4.9 (SDA)
- new net SD5_2.8: Q1.2 (S), R16.2, U6.9 (SDA)
- no-connect marks 0 -> 10
Other:
- moved on the sheet: C7, R12
